File: prototype/schematics/helios_artemis.kicad_pcb (KiCad board)
At the start: 2 copper layers, 140 x 110 mm, 4 parts

Commit message: Replace TSL2591 sensor with GY302 (BH1750) across firmware, docs, and schematics
Other:
- board text added: "SENSOR ZONE BOARD EDGE: U6 GY302 unobstructed sky view U3 INA219 C5"
- board text removed: "SENSOR ZONE BOARD EDGE: U6 TSL2591 unobstructed sky view U3 INA219 C5"
Changed lines of the file:
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@@
     (layer "Cmts.User")
   )
-  (gr_text "SENSOR ZONE BOARD EDGE: U6 TSL2591 unobstructed sky view U3 INA219 C5"
+  (gr_text "SENSOR ZONE BOARD EDGE: U6 GY302 unobstructed sky view U3 INA219 C5"
     (at 12 84 0)
     (layer "Cmts.User")
